Commit message: changed Paths

File: SCARA_4/urdf/SCARA_test.urdf (robot description, URDF)
Before this commit: robot scara, 7 links, 6 joints
Links:
- link base_link: geometry collision mesh filename=package://scara_4/meshes/base_link.STL; visual mesh filename=package://scara_4/meshes/base_link.STL
- link link_1: geometry collision mesh filename=package://scara_4/meshes/link_1.STL; visual mesh filename=package://scara_4/meshes/link_1.STL
- link link_2: geometry collision mesh filename=package://scara_4/meshes/link_2.STL; visual mesh filename=package://scara_4/meshes/link_2.STL
- link link_3: geometry collision mesh filename=package://scara_4/meshes/link_3.STL; visual mesh filename=package://scara_4/meshes/link_3.STL
- link link_4: geometry collision mesh filename=package://scara_4/meshes/link_4.STL; visual mesh filename=package://scara_4/meshes/link_4.STL
- link tool: geometry collision mesh filename=package://scara_4/meshes/tool.STL; visual mesh filename=package://scara_4/meshes/tool.STL

File: robot_arm_6dof_assembly/urdf/robot_test.urdf (robot description, URDF)
Before this commit: robot knickarm_6dof, 8 links, 7 joints
Links:
- link base_link: geometry collision mesh filename=package://robot_arm_6dof_assembly/meshes/base_link.STL; visual mesh filename=package://robot_arm_6dof_assembly/meshes/base_link.STL
- link link_1: geometry collision mesh filename=package://robot_arm_6dof_assembly/meshes/link_1.STL; visual mesh filename=package://robot_arm_6dof_assembly/meshes/link_1.STL
- link link_2: geometry collision mesh filename=package://robot_arm_6dof_assembly/meshes/link_2.STL; visual mesh filename=package://robot_arm_6dof_assembly/meshes/link_2.STL
- link link_3: geometry collision mesh filename=package://robot_arm_6dof_assembly/meshes/link_3.STL; visual mesh filename=package://robot_arm_6dof_assembly/meshes/link_3.STL
- link link_4: geometry collision mesh filename=package://robot_arm_6dof_assembly/meshes/link_4.STL; visual mesh filename=package://robot_arm_6dof_assembly/meshes/link_4.STL
- link link_5: geometry collision mesh filename=package://robot_arm_6dof_assembly/meshes/link_5.STL; visual mesh filename=package://robot_arm_6dof_assembly/meshes/link_5.STL
- link tool: geometry collision mesh filename=package://robot_arm_6dof_assembly/meshes/tool.STL; visual mesh filename=package://robot_arm_6dof_assembly/meshes/tool.STL
