Commit message: add movit

File: SCARA_4/urdf/SCARA_4.urdf (robot description, URDF)
Before this commit: robot scara, 7 links, 6 joints
Links:
- link base_link: geometry collision mesh filename=package://scara_4/meshes/base_link.STL; visual mesh filename=package://scara_4/meshes/base_link.STL
- link link_1: geometry collision mesh filename=package://scara_4/meshes/link_1.STL; visual mesh filename=package://scara_4/meshes/link_1.STL
- link link_2: geometry collision mesh filename=package://scara_4/meshes/link_2.STL; visual mesh filename=package://scara_4/meshes/link_2.STL
- link link_3: geometry collision mesh filename=package://scara_4/meshes/link_3.STL; visual mesh filename=package://scara_4/meshes/link_3.STL
- link link_4: geometry collision mesh filename=package://scara_4/meshes/link_4.STL; visual mesh filename=package://scara_4/meshes/link_4.STL
- link tool: geometry collision mesh filename=package://scara_4/meshes/tool.STL; visual mesh filename=package://scara_4/meshes/tool.STL
Joints:
- joint joint_3: limit lower=0.0 upper=0.20 effort=100.0 velocity=0.5 -> lower=-0.40 upper=0.0 effort=100.0 velocity=0.5
- joint world_to_base: origin xyz=0 0 0 rpy=1.5708 0 0 -> xyz=0 0 0 rpy=-1.5708 0 0

File: SCARA_4/urdf/SCARA_test.urdf (robot description, URDF)
Before this commit: robot scara, 7 links, 6 joints
Joints:
- joint joint_3: limit lower=0.0 upper=0.20 effort=100.0 velocity=0.5 -> lower=-0.40 upper=0.0 effort=100.0 velocity=0.5

File: SCARA_4/urdf/_SCARA_4.urdf (robot description, URDF)
Before this commit: robot SCARA_4, 6 links, 5 joints
Links:
- link base_link: geometry collision mesh filename=package://scara_4/meshes/base_link.STL; visual mesh filename=package://scara_4/meshes/base_link.STL
- link link_1: geometry collision mesh filename=package://scara_4/meshes/link_1.STL; visual mesh filename=package://scara_4/meshes/link_1.STL
- link link_2: geometry collision mesh filename=package://scara_4/meshes/link_2.STL; visual mesh filename=package://scara_4/meshes/link_2.STL
- link link_3: geometry collision mesh filename=package://scara_4/meshes/link_3.STL; visual mesh filename=package://scara_4/meshes/link_3.STL
- link link_4: geometry collision mesh filename=package://scara_4/meshes/link_4.STL; visual mesh filename=package://scara_4/meshes/link_4.STL
- link tool: geometry collision mesh filename=package://scara_4/meshes/tool.STL; visual mesh filename=package://scara_4/meshes/tool.STL
